Commit message: fix: change arm_id for prefix

File: robots/panda.gazebo.xacro (robot description, xacro)
@@ -1,39 +1,39 @@
 <?xml version="1.0"?>
 <robot xmlns:xacro="http://www.ros.org/wiki/xacro">
-    <xacro:macro name="panda_gazebo" params="robot_name load_gripper">
-      <gazebo reference="${robot_name}_joint7">
+    <xacro:macro name="panda_gazebo" params="prefix load_gripper">
+      <gazebo reference="${prefix}_joint7">
         <implicitSpringDamper>1</implicitSpringDamper>
         <provideFeedback>true</provideFeedback>
       </gazebo>
-      <gazebo reference="${robot_name}_joint1">
+      <gazebo reference="${prefix}_joint1">
         <implicitSpringDamper>1</implicitSpringDamper>
         <provideFeedback>true</provideFeedback>
       </gazebo>
-      <gazebo reference="${robot_name}_joint2">
+      <gazebo reference="${prefix}_joint2">
         <implicitSpringDamper>1</implicitSpringDamper>
         <provideFeedback>true</provideFeedback>
       </gazebo>
-      <gazebo reference="${robot_name}_joint3">
+      <gazebo reference="${prefix}_joint3">
         <implicitSpringDamper>1</implicitSpringDamper>
         <provideFeedback>true</provideFeedback>
       </gazebo>
-      <gazebo reference="${robot_name}_joint4">
+      <gazebo reference="${prefix}_joint4">
         <implicitSpringDamper>1</implicitSpringDamper>
         <provideFeedback>true</provideFeedback>
       </gazebo>
-      <gazebo reference="${robot_name}_joint5">
+      <gazebo reference="${prefix}_joint5">
         <implicitSpringDamper>1</implicitSpringDamper>
         <provideFeedback>true</provideFeedback>
       </gazebo>
-      <gazebo reference="${robot_name}_joint6">
+      <gazebo reference="${prefix}_joint6">
         <implicitSpringDamper>1</implicitSpringDamper>
         <provideFeedback>true</provideFeedback>
       </gazebo>
       <xacro:if value="${load_gripper}">
-          <gazebo reference="${robot_name}_finger_joint1">
+          <gazebo reference="${prefix}_finger_joint1">
             <implicitSpringDamper>1</implicitSpringDamper>
             <provideFeedback>true</provideFeedback>
           </gazebo>
-          <gazebo reference="${robot_name}_finger_joint2">
+          <gazebo reference="${prefix}_finger_joint2">
             <implicitSpringDamper>1</implicitSpringDamper>
             <provideFeedback>true</provideFeedback>
@@ -41,7 +41,7 @@
       </xacro:if>
     <!-- Adding FT sensor at wrist. This is not present in real robot and is used only for computing end-point effort directly, unlike in the real robot where it is estimated from the joint efforts. -->
-    <gazebo reference="${robot_name}_joint7">
+    <gazebo reference="${prefix}_joint7">
       <disableFixedJointLumping>true</disableFixedJointLumping>
-      <sensor name="${robot_name}_joint7_force_torque" type="force_torque">
+      <sensor name="${prefix}_joint7_force_torque" type="force_torque">
         <always_on>true</always_on>
         <visualize>false</visualize>

File: robots/panda_arm.urdf.xacro (robot description, xacro)
@@ -2,5 +2,5 @@
 <robot xmlns:xacro="http://www.ros.org/wiki/xacro" name="panda">
     <xacro:arg name="load_gazebo" default="false"/>
-    <xacro:arg name="arm_id" default="panda"/>
+    <xacro:arg name="prefix" default="panda"/>
     <xacro:arg name="connected_to" default=""/>
     <xacro:arg name="xyz" default="0 0 0"/>
@@ -10,9 +10,9 @@
     <xacro:include filename="$(find franka_panda_description)/ros2_control/panda_arm.ros2_control.xacro"/>
     <xacro:if value="$(arg load_gazebo)">
-        <xacro:panda_arm arm_id="$(arg arm_id)" connected_to="$(arg connected_to)" xyz="$(arg xyz)" rpy="$(arg rpy)" in_gazebo="true"/>
+        <xacro:panda_arm prefix="$(arg prefix)" connected_to="$(arg connected_to)" xyz="$(arg xyz)" rpy="$(arg rpy)" in_gazebo="true"/>
     </xacro:if>
     <xacro:unless value="$(arg load_gazebo)">
-        <xacro:panda_arm arm_id="$(arg arm_id)" connected_to="$(arg connected_to)" xyz="$(arg xyz)" rpy="$(arg rpy)"/>
+        <xacro:panda_arm prefix="$(arg prefix)" connected_to="$(arg connected_to)" xyz="$(arg xyz)" rpy="$(arg rpy)"/>
     </xacro:unless>
-    <xacro:panda_arm_interface name="PandaInterface" arm_id="$(arg arm_id)"/>
+    <xacro:panda_arm_interface name="PandaInterface" prefix="$(arg prefix)"/>
 </robot>

File: robots/panda_arm.xacro (robot description, xacro)
@@ -1,5 +1,5 @@
 <?xml version='1.0'?>
 <robot xmlns:xacro="http://www.ros.org/wiki/xacro" name="panda">
-  <xacro:macro name="panda_arm" params="arm_id:='panda' description_pkg:='franka_panda_description' connected_to:='' in_gazebo='false' xyz:='0 0 0' rpy:='0 0 0'">
+  <xacro:macro name="panda_arm" params="prefix:='panda' description_pkg:='franka_panda_description' connected_to:='' in_gazebo='false' xyz:='0 0 0' rpy:='0 0 0'">
     <!-- If using custom frame with ${connected_to} param, make sure 'world' frame exists in its TF tree -->
     <xacro:if value="${connected_to == ''}">
@@ -10,7 +10,7 @@
       <xacro:property name="base_frame_name" value="${connected_to}"/>
     </xacro:unless>
-    <joint name="${arm_id}_to_${base_frame_name}" type="fixed">
+    <joint name="${prefix}_to_${base_frame_name}" type="fixed">
       <parent link="${base_frame_name}"/>
-      <child link="${arm_id}_link0"/>
+      <child link="${prefix}_link0"/>
       <origin rpy="${rpy}" xyz="${xyz}"/>
       <xacro:unless value="${in_gazebo == 'false'}">
@@ -18,5 +18,5 @@
       </xacro:unless>
     </joint>
-    <link name="${arm_id}_link0">
+    <link name="${prefix}_link0">
       <visual>
         <geometry>
@@ -37,5 +37,5 @@
       </xacro:unless>
     </link>
-    <link name="${arm_id}_link1">
+    <link name="${prefix}_link1">
       <visual>
         <geometry>
@@ -54,14 +54,14 @@
       </inertial>
     </link>
-    <joint name="${arm_id}_joint1" type="revolute">
+    <joint name="${prefix}_joint1" type="revolute">
       <safety_controller k_position="100.0" k_velocity="40.0" soft_lower_limit="-2.8973" soft_upper_limit="2.8973"/>
       <origin rpy="0 0 0" xyz="0 0 0.333"/>
-      <parent link="${arm_id}_link0"/>
-      <child link="${arm_id}_link1"/>
+      <parent link="${prefix}_link0"/>
+      <child link="${prefix}_link1"/>
       <axis xyz="0 0 1"/>
       <limit effort="87" lower="-2.8973" upper="2.8973" velocity="2.1750"/>
       <dynamics damping="10.0" friction="5.0"/>
     </joint>
-    <link name="${arm_id}_link2">
+    <link name="${prefix}_link2">
       <visual>
         <geometry>
@@ -80,14 +80,14 @@
       </inertial>
     </link>
-    <joint name="${arm_id}_joint2" type="revolute">
+    <joint name="${prefix}_joint2" type="revolute">
       <safety_controller k_position="100.0" k_velocity="40.0" soft_lower_limit="-1.7628" soft_upper_limit="1.7628"/>
       <origin rpy="${-pi/2} 0 0" xyz="0 0 0"/>
-      <parent link="${arm_id}_link1"/>
-      <child link="${arm_id}_link2"/>
+      <parent link="${prefix}_link1"/>
+      <child link="${prefix}_link2"/>
       <axis xyz="0 0 1"/>
       <limit effort="87" lower="-1.7628" upper="1.7628" velocity="2.1750"/>
       <dynamics damping="5.0" friction="2.0"/>
     </joint>
-    <link name="${arm_id}_link3">
+    <link name="${prefix}_link3">
       <visual>
         <geometry>
@@ -106,14 +106,14 @@
       </inertial>
     </link>
-    <joint name="${arm_id}_joint3" type="revolute">
+    <joint name="${prefix}_joint3" type="revolute">
       <safety_controller k_position="100.0" k_velocity="40.0" soft_lower_limit="-2.8973" soft_upper_limit="2.8973"/>
       <origin rpy="${pi/2} 0 0" xyz="0 -0.316 0"/>
-      <parent link="${arm_id}_link2"/>
-      <child link="${arm_id}_link3"/>
+      <parent link="${prefix}_link2"/>
+      <child link="${prefix}_link3"/>
       <axis xyz="0 0 1"/>
       <limit effort="87" lower="-2.8973" upper="2.8973" velocity="2.1750"/>
       <dynamics damping="5.0" friction="2.0"/>
     </joint>
-    <link name="${arm_id}_link4">
+    <link name="${prefix}_link4">
       <visual>
         <geometry>
@@ -132,14 +132,14 @@
       </inertial>
     </link>
-    <joint name="${arm_id}_joint4" type="revolute">
+    <joint name="${prefix}_joint4" type="revolute">
       <safety_controller k_position="100.0" k_velocity="40.0" soft_lower_limit="-3.0718" soft_upper_limit="-0.0698"/>
       <origin rpy="${pi/2} 0 0" xyz="0.0825 0 0"/>
-      <parent link="${arm_id}_link3"/>
-      <child link="${arm_id}_link4"/>
+      <parent link="${prefix}_link3"/>
+      <child link="${prefix}_link4"/>
       <axis xyz="0 0 1"/>
       <limit effort="87" lower="-3.0718" upper="-0.0698" velocity="2.1750"/>
       <dynamics damping="1.0" friction="0.5"/>
     </joint>
-    <link name="${arm_id}_link5">
+    <link name="${prefix}_link5">
       <visual>
         <geometry>
@@ -158,14 +158,14 @@
       </inertial>
     </link>
-    <joint name="${arm_id}_joint5" type="revolute">
+    <joint name="${prefix}_joint5" type="revolute">
       <safety_controller k_position="100.0" k_velocity="40.0" soft_lower_limit="-2.8973" soft_upper_limit="2.8973"/>
       <origin rpy="${-pi/2} 0 0" xyz="-0.0825 0.384 0"/>
-      <parent link="${arm_id}_link4"/>
-      <child link="${arm_id}_link5"/>
+      <parent link="${prefix}_link4"/>
+      <child link="${prefix}_link5"/>
       <axis xyz="0 0 1"/>
       <limit effort="12" lower="-2.8973" upper="2.8973" velocity="2.6100"/>
       <dynamics damping="2.0" friction="1.0"/>
     </joint>
-    <link name="${arm_id}_link6">
+    <link name="${prefix}_link6">
       <visual>
         <geometry>
@@ -184,14 +184,14 @@
       </inertial>
     </link>
-    <joint name="${arm_id}_joint6" type="revolute">
+    <joint name="${prefix}_joint6" type="revolute">
       <safety_controller k_position="100.0" k_velocity="40.0" soft_lower_limit="-0.0175" soft_upper_limit="3.7525"/>
       <origin rpy="${pi/2} 0 0" xyz="0 0 0"/>
-      <parent link="${arm_id}_link5"/>
-      <child link="${arm_id}_link6"/>
+      <parent link="${prefix}_link5"/>
+      <child link="${prefix}_link6"/>
       <axis xyz="0 0 1"/>
       <limit effort="12" lower="-0.0175" upper="3.7525" velocity="2.6100"/>
       <dynamics damping="1.0" friction="0.5"/>
     </joint>
-    <link name="${arm_id}_link7">
+    <link name="${prefix}_link7">
       <visual>
         <geometry>
@@ -210,14 +210,14 @@
       </inertial>
     </link>
-    <joint name="${arm_id}_joint7" type="revolute">
+    <joint name="${prefix}_joint7" type="revolute">
       <safety_controller k_position="100.0" k_velocity="40.0" soft_lower_limit="-2.8973" soft_upper_limit="2.8973"/>
       <origin rpy="${pi/2} 0 0" xyz="0.088 0 0"/>
-      <parent link="${arm_id}_link6"/>
-      <child link="${arm_id}_link7"/>
+      <parent link="${prefix}_link6"/>
+      <child link="${prefix}_link7"/>
       <axis xyz="0 0 1"/>
       <limit effort="12" lower="-2.8973" upper="2.8973" velocity="2.6100"/>
       <dynamics damping="1.0" friction="0.5"/>
     </joint>
-    <link name="${arm_id}_link8">
+    <link name="${prefix}_link8">
       <inertial>
         <origin xyz="0 0 0" rpy="0 0 0"/>
@@ -226,8 +226,8 @@
       </inertial>
     </link>
-    <joint name="${arm_id}_joint8" type="fixed">
+    <joint name="${prefix}_joint8" type="fixed">
     <origin rpy="0 0 0" xyz="0 0 0.107"/>
-      <parent link="${arm_id}_link7"/>
-      <child link="${arm_id}_link8"/>
+      <parent link="${prefix}_link7"/>
+      <child link="${prefix}_link8"/>
       <axis xyz="0 0 0"/>
     </joint>

File: ros2_control/panda_arm.ros2_control.xacro (robot description, xacro)
@@ -1,10 +1,10 @@
 <?xml version="1.0"?>
 <robot xmlns:xacro="http://www.ros.org/wiki/xacro">
-  <xacro:macro name="panda_arm_interface" params="name arm_id:='panda'">
+  <xacro:macro name="panda_arm_interface" params="name prefix:='panda'">
     <hardware>
       <plugin>robot_interface/franka/PandaInterface</plugin>
     </hardware>
     <ros2_control name="${name}" type="system">
-      <joint name="${arm_id}_joint1">
+      <joint name="${prefix}_joint1">
         <command_interface name="position">
           <param name="min">-2.8973</param>
@@ -24,5 +24,5 @@
         <state_interface name="effort"/>
       </joint>
-      <joint name="${arm_id}_joint2">
+      <joint name="${prefix}_joint2">
         <command_interface name="position">
           <param name="min">-1.7628</param>
@@ -42,5 +42,5 @@
         <state_interface name="effort"/>
       </joint>
-      <joint name="${arm_id}_joint3">
+      <joint name="${prefix}_joint3">
         <command_interface name="position">
           <param name="min">-2.8973</param>
@@ -60,5 +60,5 @@
         <state_interface name="effort"/>
       </joint>
-      <joint name="${arm_id}_joint4">
+      <joint name="${prefix}_joint4">
         <command_interface name="position">
           <param name="min">-3.0718</param>
@@ -78,5 +78,5 @@
         <state_interface name="effort"/>
       </joint>
-      <joint name="${arm_id}_joint5">
+      <joint name="${prefix}_joint5">
         <command_interface name="position">
           <param name="min">-2.8973</param>
@@ -96,5 +96,5 @@
         <state_interface name="effort"/>
       </joint>
-      <joint name="${arm_id}_joint6">
+      <joint name="${prefix}_joint6">
         <command_interface name="position">
           <param name="min">-0.0175</param>
@@ -114,5 +114,5 @@
         <state_interface name="effort"/>
       </joint>
-      <joint name="${arm_id}_joint7">
+      <joint name="${prefix}_joint7">
         <command_interface name="position">
           <param name="min">-2.8973</param>
