Commit message: fix: correctly include the ros2_control macro

File: robots/panda_arm.urdf.xacro (robot description, xacro)
@@ -10,8 +10,9 @@
     <xacro:include filename="$(find franka_panda_description)/ros2_control/panda_arm.ros2_control.xacro"/>
     <xacro:if value="$(arg load_gazebo)">
-        <xacro:panda_arm arm_id="$(arg arm_id)" connected_to="$(arg connected_to)" xyz="$(arg xyz)" rpy="$(arg rpy)" in_gazebo="true" />
+        <xacro:panda_arm arm_id="$(arg arm_id)" connected_to="$(arg connected_to)" xyz="$(arg xyz)" rpy="$(arg rpy)" in_gazebo="true"/>
     </xacro:if>
     <xacro:unless value="$(arg load_gazebo)">
-        <xacro:panda_arm arm_id="$(arg arm_id)" connected_to="$(arg connected_to)" xyz="$(arg xyz)" rpy="$(arg rpy)" />
+        <xacro:panda_arm arm_id="$(arg arm_id)" connected_to="$(arg connected_to)" xyz="$(arg xyz)" rpy="$(arg rpy)"/>
     </xacro:unless>
+    <xacro:panda_arm_interface name="PandaInterface" arm_id="$(arg arm_id)"/>
 </robot>

File: ros2_control/panda_arm.ros2_control.xacro (robot description, xacro)
@@ -1,5 +1,5 @@
 <?xml version="1.0"?>
 <robot xmlns:xacro="http://www.ros.org/wiki/xacro">
-  <xacro:macro name="panda_arm" params="name prefix arm_id:='panda">
+  <xacro:macro name="panda_arm_interface" params="name arm_id:='panda'">
     <hardware>
       <plugin>robot_interface/franka/PandaInterface</plugin>

Commit message: fix: correct typo in the macros

File: robots/panda_arm.urdf.xacro (robot description, xacro)
@@ -2,5 +2,5 @@
 <robot xmlns:xacro="http://www.ros.org/wiki/xacro" name="panda">
     <xacro:arg name="load_gazebo" default="false"/>
-    <xacro:arg name="prefix" default="panda"/>
+    <xacro:arg name="prefix" default="panda_"/>
     <xacro:arg name="use_sim" default="false"/>
     <xacro:arg name="connected_to" default=""/>
@@ -16,4 +16,4 @@
         <xacro:panda_arm prefix="$(arg prefix)" connected_to="$(arg connected_to)" xyz="$(arg xyz)" rpy="$(arg rpy)"/>
     </xacro:unless>
-    <xacro:panda_arm_interface name="PandaInterface" prefix="$(arg prefix) use_sim="$(arg use_sim)"/>
+    <xacro:panda_arm_interface name="PandaInterface" prefix="$(arg prefix)" use_sim="$(arg use_sim)"/>
 </robot>

File: ros2_control/panda_arm.ros2_control.xacro (robot description, xacro)
@@ -1,14 +1,16 @@
 <?xml version="1.0"?>
 <robot xmlns:xacro="http://www.ros.org/wiki/xacro">
-  <xacro:macro name="panda_arm_interface" params="name prefix:='panda_' use_sim:=^|false">
+  <xacro:macro name="panda_arm_interface" params="name prefix use_sim:=^|false">
     <ros2_control name="${name}" type="system">
-      <hardware>
-        <xacro:if value="$(arg use_sim)">
+      <xacro:if value="$(arg use_sim)">
+        <hardware>
           <plugin>robot_interface/simulators/PybulletInterface</plugin>
-        </xacro:if>
-        <xacro:unless value="$(arg use_sim)">
+        </hardware>
+      </xacro:if>
+      <xacro:unless value="$(arg use_sim)">
+        <hardware>
           <plugin>robot_interface/franka/PandaInterface</plugin>
-        </xacro:unless>
-      </hardware>
+        </hardware>
+      </xacro:unless>
       <joint name="${prefix}joint1">
         <command_interface name="position">

Commit message: Add simulation tag (#4)

File: robots/panda_arm.urdf.xacro (robot description, xacro)
@@ -2,5 +2,6 @@
 <robot xmlns:xacro="http://www.ros.org/wiki/xacro" name="panda">
     <xacro:arg name="load_gazebo" default="false"/>
-    <xacro:arg name="prefix" default="panda"/>
+    <xacro:arg name="prefix" default="panda_"/>
+    <xacro:arg name="use_sim" default="false"/>
     <xacro:arg name="connected_to" default=""/>
     <xacro:arg name="xyz" default="0 0 0"/>
@@ -15,4 +16,4 @@
         <xacro:panda_arm prefix="$(arg prefix)" connected_to="$(arg connected_to)" xyz="$(arg xyz)" rpy="$(arg rpy)"/>
     </xacro:unless>
-    <xacro:panda_arm_interface name="PandaInterface" prefix="$(arg prefix)"/>
+    <xacro:panda_arm_interface name="PandaInterface" prefix="$(arg prefix)" use_sim="$(arg use_sim)"/>
 </robot>

File: ros2_control/panda_arm.ros2_control.xacro (robot description, xacro)
@@ -1,9 +1,16 @@
 <?xml version="1.0"?>
 <robot xmlns:xacro="http://www.ros.org/wiki/xacro">
-  <xacro:macro name="panda_arm_interface" params="name prefix:='panda_'">
+  <xacro:macro name="panda_arm_interface" params="name prefix use_sim:=^|false">
     <ros2_control name="${name}" type="system">
-      <hardware>
-        <plugin>robot_interface/franka/PandaInterface</plugin>
-      </hardware>
+      <xacro:if value="$(arg use_sim)">
+        <hardware>
+          <plugin>robot_interface/simulators/PybulletInterface</plugin>
+        </hardware>
+      </xacro:if>
+      <xacro:unless value="$(arg use_sim)">
+        <hardware>
+          <plugin>robot_interface/franka/PandaInterface</plugin>
+        </hardware>
+      </xacro:unless>
       <joint name="${prefix}joint1">
         <command_interface name="position">

Commit message: feat: add communication parameters in the URDF

File: robots/panda_arm.urdf.xacro (robot description, xacro)
@@ -2,4 +2,7 @@
 <robot xmlns:xacro="http://www.ros.org/wiki/xacro" name="panda">
     <xacro:arg name="prefix" default="panda_"/>
+    <xacro:arg name="robot_ip" default="127.0.0.1"/>
+    <xacro:arg name="robot_state_port" default="1601"/>
+    <xacro:arg name="robot_command_port" default="1602"/>
     <xacro:arg name="load_gazebo" default="false"/>
     <xacro:arg name="load_ros2_control" default="false"/>
@@ -18,5 +21,12 @@
     </xacro:unless>
     <xacro:if value="$(arg load_ros2_control)">
-        <xacro:panda_arm_interface name="PandaInterface" prefix="$(arg prefix)" use_sim="$(arg use_sim)"/>
+        <xacro:panda_arm_interface
+                name="PandaInterface"
+                prefix="$(arg prefix)"
+                robot_ip="$(arg robot_ip)"
+                robot_state_port="$(arg robot_state_port)"
+                robot_command_port="$(arg robot_command_port)"
+                use_sim="$(arg use_sim)"
+        />
     </xacro:if>
 </robot>

File: ros2_control/panda_arm.ros2_control.xacro (robot description, xacro)
@@ -1,14 +1,20 @@
 <?xml version="1.0"?>
 <robot xmlns:xacro="http://www.ros.org/wiki/xacro">
-  <xacro:macro name="panda_arm_interface" params="name prefix use_sim:=^|false">
+  <xacro:macro name="panda_arm_interface" params="name prefix robot_ip robot_state_port robot_command_port use_sim">
     <ros2_control name="${name}" type="system">
-      <xacro:if value="$(arg use_sim)">
+      <xacro:if value="${use_sim}">
         <hardware>
           <plugin>robot_interface/simulators/PybulletInterface</plugin>
+          <param name="robot_ip">${robot_ip}</param>
+          <param name="robot_state_port">${robot_state_port}</param>
+          <param name="robot_command_port">${robot_command_port}</param>
         </hardware>
       </xacro:if>
-      <xacro:unless value="$(arg use_sim)">
+      <xacro:unless value="${use_sim}">
         <hardware>
           <plugin>robot_interface/franka/PandaInterface</plugin>
+          <param name="robot_ip">${robot_ip}</param>
+          <param name="robot_state_port">${robot_state_port}</param>
+          <param name="robot_command_port">"${robot_command_port}</param>
         </hardware>
       </xacro:unless>
