Commit message: Use prefix argument in hand xacro too

File: robots/hand.urdf.xacro (robot description, xacro)
@@ -2,4 +2,4 @@
 <robot xmlns:xacro="http://www.ros.org/wiki/xacro" name="hand">
   <xacro:include filename="hand.xacro"/>
-  <xacro:hand ns="panda"/>
+  <xacro:hand/>
 </robot>

File: robots/hand.xacro (robot description, xacro)
@@ -1,13 +1,13 @@
 <?xml version="1.0" encoding="utf-8"?>
 <robot xmlns:xacro="http://www.ros.org/wiki/xacro" name="hand">
-  <xacro:macro name="hand" params="connected_to:='' ns:='' rpy:='0 0 0' xyz:='0 0 0' ">
+  <xacro:macro name="hand" params="connected_to:='' prefix:='panda_' rpy:='0 0 0' xyz:='0 0 0' ">
     <xacro:unless value="${connected_to == ''}">
-      <joint name="${ns}_hand_joint" type="fixed">
+      <joint name="${prefix}hand_joint" type="fixed">
         <parent link="${connected_to}"/>
-        <child link="${ns}_hand"/>
+        <child link="${prefix}hand"/>
         <origin xyz="${xyz}" rpy="${rpy}"/>
       </joint>
     </xacro:unless>
-    <link name="${ns}_hand">
+    <link name="${prefix}hand">
       <visual>
         <geometry>
@@ -26,5 +26,5 @@
       </inertial>
     </link>
-    <link name="${ns}_leftfinger">
+    <link name="${prefix}leftfinger">
       <visual>
         <geometry>
@@ -43,5 +43,5 @@
       </inertial>
     </link>
-    <link name="${ns}_rightfinger">
+    <link name="${prefix}rightfinger">
       <visual>
         <origin xyz="0 0 0" rpy="0 0 ${pi}"/>
@@ -62,7 +62,7 @@
       </inertial>
     </link>
-    <joint name="${ns}_finger_joint1" type="prismatic">
-      <parent link="${ns}_hand"/>
-      <child link="${ns}_leftfinger"/>
+    <joint name="${prefix}finger_joint1" type="prismatic">
+      <parent link="${prefix}hand"/>
+      <child link="${prefix}leftfinger"/>
       <origin xyz="0 0 0.0584" rpy="0 0 0"/>
       <axis xyz="0 1 0"/>
@@ -70,12 +70,12 @@
       <dynamics damping="500.0" friction="0.0"/>
     </joint>
-    <joint name="${ns}_finger_joint2" type="prismatic">
-      <parent link="${ns}_hand"/>
-      <child link="${ns}_rightfinger"/>
+    <joint name="${prefix}finger_joint2" type="prismatic">
+      <parent link="${prefix}hand"/>
+      <child link="${prefix}rightfinger"/>
       <origin xyz="0 0 0.0584" rpy="0 0 0"/>
       <axis xyz="0 -1 0"/>
       <limit effort="20" lower="0.0" upper="0.04" velocity="0.2"/>
       <dynamics damping="500.0" friction="0.0"/>
-      <mimic joint="${ns}_finger_joint1" />
+      <mimic joint="${prefix}finger_joint1"/>
     </joint>
   </xacro:macro>

File: robots/panda_arm_hand.urdf.xacro (robot description, xacro)
@@ -1,5 +1,5 @@
 <?xml version="1.0"?>
 <robot xmlns:xacro="http://www.ros.org/wiki/xacro" name="panda">
-  <xacro:arg name="robot_name" default="panda"/>
+  <xacro:arg name="prefix" default="panda_"/>
   <xacro:arg name="load_gripper" default="true"/>
   <xacro:arg name="connected_to" default=""/>
@@ -7,5 +7,5 @@
   <xacro:if value="$(arg load_gripper)">
     <xacro:include filename="$(find franka_panda_description)/robots/hand.xacro"/>
-    <xacro:hand ns="panda" rpy="0 0 ${-pi/4}" connected_to="panda_link8"/>
+    <xacro:hand prefix="$(arg prefix)" rpy="0 0 ${-pi/4}" connected_to="$(arg prefix)link8"/>
   </xacro:if>
   <xacro:panda_arm prefix="$(arg prefix)" connected_to="$(arg connected_to)"/>

Commit message: Fix hand urdf xacro

File: robots/hand.urdf.xacro (robot description, xacro)
@@ -2,13 +2,18 @@
 <robot xmlns:xacro="http://www.ros.org/wiki/xacro" name="hand">
   <xacro:arg name="prefix" default="panda_"/>
-  <xacro:arg name="robot_ip" default="172.16.0.2"/>
-  <xacro:arg name="load_ros2_control" default="false"/>
+  <xacro:arg name="connected_to" default=""/>
   <xacro:arg name="fix_finger_joints" default="false"/>
   <xacro:arg name="insert_grasp_frame" default="false"/>
-  <xacro:arg name="connected_to" default=""/>
+  <xacro:arg name="load_ros2_control" default="false"/>
+  <xacro:arg name="robot_ip" default="172.16.0.2"/>
+  <xacro:arg name="use_sim" default="false"/>
   <xacro:arg name="xyz" default="0 0 0"/>
-  <xacro:arg name="rpy" default="0 0 0"/>
+  <xacro:arg name="rpy" default="0 0 -0.785398"/>
   <xacro:include filename="hand.xacro"/>
-  <xacro:hand prefix="$(arg prefix)" connected_to="$(arg connected_to)" xyz="$(arg xyz)" rpy="$(arg rpy)"
+  <xacro:property name="connected_to" value="$(arg connected_to)"/>
+  <xacro:unless value="${connected_to == ''}">
+    <link name="${connected_to}"/>
+  </xacro:unless>
+  <xacro:hand prefix="$(arg prefix)" connected_to="${connected_to}" xyz="$(arg xyz)" rpy="$(arg rpy)"
               fix_finger_joints="$(arg fix_finger_joints)" insert_grasp_frame="$(arg insert_grasp_frame)"/>
   <xacro:unless value="$(arg fix_finger_joints)">
