Commit message: Add option to fix finger joints and insert grasp frame

File: robots/hand.xacro (robot description, xacro)
@@ -1,5 +1,6 @@
 <?xml version="1.0" encoding="utf-8"?>
 <robot xmlns:xacro="http://www.ros.org/wiki/xacro" name="hand">
-  <xacro:macro name="hand" params="connected_to:='' prefix:='panda_' rpy:='0 0 0' xyz:='0 0 0' ">
+  <xacro:macro name="hand"
+               params="prefix:='panda_' connected_to:='' rpy:='0 0 0' xyz:='0 0 0' fix_finger_joints=false insert_grasp_frame:=false">
     <xacro:unless value="${connected_to == ''}">
       <joint name="${prefix}hand_joint" type="fixed">
@@ -62,21 +63,43 @@
       </inertial>
     </link>
-    <joint name="${prefix}finger_joint1" type="prismatic">
-      <parent link="${prefix}hand"/>
-      <child link="${prefix}leftfinger"/>
-      <origin xyz="0 0 0.0584" rpy="0 0 0"/>
-      <axis xyz="0 1 0"/>
-      <limit effort="20" lower="0.0" upper="0.04" velocity="0.2"/>
-      <dynamics damping="500.0" friction="0.0"/>
-    </joint>
-    <joint name="${prefix}finger_joint2" type="prismatic">
-      <parent link="${prefix}hand"/>
-      <child link="${prefix}rightfinger"/>
-      <origin xyz="0 0 0.0584" rpy="0 0 0"/>
-      <axis xyz="0 -1 0"/>
-      <limit effort="20" lower="0.0" upper="0.04" velocity="0.2"/>
-      <dynamics damping="500.0" friction="0.0"/>
-      <mimic joint="${prefix}finger_joint1"/>
-    </joint>
+    <xacro:unless value="${fix_finger_joints}">
+      <joint name="${prefix}finger_joint1" type="prismatic">
+        <parent link="${prefix}hand"/>
+        <child link="${prefix}leftfinger"/>
+        <origin xyz="0 0 0.0584" rpy="0 0 0"/>
+        <axis xyz="0 1 0"/>
+        <limit effort="20" lower="0.0" upper="0.04" velocity="0.2"/>
+        <dynamics damping="500.0" friction="0.0"/>
+      </joint>
+      <joint name="${prefix}finger_joint2" type="prismatic">
+        <parent link="${prefix}hand"/>
+        <child link="${prefix}rightfinger"/>
+        <origin xyz="0 0 0.0584" rpy="0 0 0"/>
+        <axis xyz="0 -1 0"/>
+        <limit effort="20" lower="0.0" upper="0.04" velocity="0.2"/>
+        <dynamics damping="500.0" friction="0.0"/>
+        <mimic joint="${prefix}finger_joint1"/>
+      </joint>
+    </xacro:unless>
+    <xacro:if value="${fix_finger_joints}">
+      <joint name="${prefix}finger_joint1" type="fixed">
+        <parent link="${prefix}hand"/>
+        <child link="${prefix}leftfinger"/>
+        <origin xyz="0 0.04 0.0584" rpy="0 0 0"/>
+      </joint>
+      <joint name="${prefix}finger_joint2" type="fixed">
+        <parent link="${prefix}hand"/>
+        <child link="${prefix}rightfinger"/>
+        <origin xyz="0 -0.04 0.0584" rpy="0 0 0"/>
+      </joint>
+    </xacro:if>
+    <xacro:if value="${insert_grasp_frame}">
+      <joint name="${prefix}_grasp_frame" type="fixed">
+        <parent link="${prefix}hand"/>
+        <child link="${prefix}hand_grasp"/>
+        <origin xyz="0 0 0.1034" rpy="0 0 0"/>
+      </joint>
+      <link name="${prefix}hand_grasp"/>
+    </xacro:if>
   </xacro:macro>
 </robot>

File: robots/panda_arm.urdf.xacro (robot description, xacro)
@@ -1,31 +1,34 @@
 <?xml version='1.0' ?>
 <robot xmlns:xacro="http://www.ros.org/wiki/xacro" name="panda">
-    <xacro:arg name="prefix" default="panda_"/>
-    <xacro:arg name="robot_ip" default="127.0.0.1"/>
-    <xacro:arg name="robot_state_port" default="1601"/>
-    <xacro:arg name="robot_command_port" default="1602"/>
-    <xacro:arg name="load_ros2_control" default="false"/>
-    <xacro:arg name="load_hand" default="false"/>
-    <xacro:arg name="use_sim" default="false"/>
-    <xacro:arg name="connected_to" default=""/>
-    <xacro:arg name="xyz" default="0 0 0"/>
-    <xacro:arg name="rpy" default="0 0 0"/>
-    <xacro:include filename="$(find franka_panda_description)/robots/panda_arm.xacro"/>
-    <!-- Import ros2_control description -->
-    <xacro:include filename="$(find franka_panda_description)/ros2_control/panda_arm.ros2_control.xacro"/>
-    <xacro:panda_arm prefix="$(arg prefix)" connected_to="$(arg connected_to)" xyz="$(arg xyz)" rpy="$(arg rpy)"/>
-    <xacro:if value="$(arg load_ros2_control)">
-        <xacro:panda_arm_interface
-                name="PandaInterface"
-                prefix="$(arg prefix)"
-                robot_ip="$(arg robot_ip)"
-                robot_state_port="$(arg robot_state_port)"
-                robot_command_port="$(arg robot_command_port)"
-                use_sim="$(arg use_sim)"
-        />
-    </xacro:if>
-    <xacro:if value="$(arg load_hand)">
-        <xacro:include filename="$(find franka_panda_description)/robots/hand.xacro"/>
-        <xacro:hand prefix="$(arg prefix)" rpy="0 0 ${-pi/4}" connected_to="$(arg prefix)link8"/>
-    </xacro:if>
+  <xacro:arg name="prefix" default="panda_"/>
+  <xacro:arg name="robot_ip" default="127.0.0.1"/>
+  <xacro:arg name="robot_state_port" default="1601"/>
+  <xacro:arg name="robot_command_port" default="1602"/>
+  <xacro:arg name="load_ros2_control" default="false"/>
+  <xacro:arg name="load_hand" default="false"/>
+  <xacro:arg name="fix_finger_joints" default="false"/>
+  <xacro:arg name="insert_grasp_frame" default="false"/>
+  <xacro:arg name="use_sim" default="false"/>
+  <xacro:arg name="connected_to" default=""/>
+  <xacro:arg name="xyz" default="0 0 0"/>
+  <xacro:arg name="rpy" default="0 0 0"/>
+  <xacro:include filename="$(find franka_panda_description)/robots/panda_arm.xacro"/>
+  <!-- Import ros2_control description -->
+  <xacro:include filename="$(find franka_panda_description)/ros2_control/panda_arm.ros2_control.xacro"/>
+  <xacro:panda_arm prefix="$(arg prefix)" connected_to="$(arg connected_to)" xyz="$(arg xyz)" rpy="$(arg rpy)"/>
+  <xacro:if value="$(arg load_ros2_control)">
+    <xacro:panda_arm_interface
+        name="PandaInterface"
+        prefix="$(arg prefix)"
+        robot_ip="$(arg robot_ip)"
+        robot_state_port="$(arg robot_state_port)"
+        robot_command_port="$(arg robot_command_port)"
+        use_sim="$(arg use_sim)"
+    />
+  </xacro:if>
+  <xacro:if value="$(arg load_hand)">
+    <xacro:include filename="$(find franka_panda_description)/robots/hand.xacro"/>
+    <xacro:hand prefix="$(arg prefix)" connected_to="$(arg prefix)link8" rpy="0 0 ${-pi/4}"
+                fix_finger_joints="$(arg fix_finger_joints)" insert_grasp_frame="$(arg insert_grasp_frame)"/>
+  </xacro:if>
 </robot>

Commit message: Clean up xacros

File: robots/hand.xacro (robot description, xacro)
@@ -1,5 +1,5 @@
 <?xml version="1.0" encoding="utf-8"?>
 <robot xmlns:xacro="http://www.ros.org/wiki/xacro" name="hand">
-  <xacro:macro name="hand" params="connected_to:='' prefix:='panda_' rpy:='0 0 0' xyz:='0 0 0' ">
+  <xacro:macro name="hand" params="prefix:='panda_' connected_to:='' xyz:='0 0 0' rpy:='0 0 0'">
     <xacro:unless value="${connected_to == ''}">
       <joint name="${prefix}hand_joint" type="fixed">

File: robots/l515_adapter.xacro (robot description, xacro)
@@ -1,6 +1,5 @@
 <?xml version="1.0" ?>
 <robot name="l515_adapter" xmlns:xacro="http://wiki.ros.org/xacro">
-  <xacro:macro name="l515_adapter"
-               params="prefix='l515_adapter_' connected_to:='' xyz:='0 0 0' rpy:='0 0 0'">
+  <xacro:macro name="l515_adapter" params="prefix='l515_adapter_' connected_to:='' xyz:='0 0 0' rpy:='0 0 0'">
     <xacro:if value="${connected_to == ''}">
       <link name="world"/>
@@ -33,5 +32,6 @@
         <origin rpy="0 0 0" xyz="0 0 0"/>
         <geometry>
-          <mesh filename="package://franka_panda_description/meshes/collision/l515_adapter.stl" scale="0.001 0.001 0.001"/>
+          <mesh filename="package://franka_panda_description/meshes/collision/l515_adapter.stl"
+                scale="0.001 0.001 0.001"/>
         </geometry>
       </collision>

File: robots/panda_arm.urdf.xacro (robot description, xacro)
@@ -1,31 +1,31 @@
-<?xml version='1.0' ?>
+<?xml version="1.0"?>
 <robot xmlns:xacro="http://www.ros.org/wiki/xacro" name="panda">
-    <xacro:arg name="prefix" default="panda_"/>
-    <xacro:arg name="robot_ip" default="127.0.0.1"/>
-    <xacro:arg name="robot_state_port" default="1601"/>
-    <xacro:arg name="robot_command_port" default="1602"/>
-    <xacro:arg name="load_ros2_control" default="false"/>
-    <xacro:arg name="load_hand" default="false"/>
-    <xacro:arg name="use_sim" default="false"/>
-    <xacro:arg name="connected_to" default=""/>
-    <xacro:arg name="xyz" default="0 0 0"/>
-    <xacro:arg name="rpy" default="0 0 0"/>
-    <xacro:include filename="$(find franka_panda_description)/robots/panda_arm.xacro"/>
+  <xacro:arg name="prefix" default="panda_"/>
+  <xacro:arg name="robot_ip" default="127.0.0.1"/>
+  <xacro:arg name="robot_state_port" default="1601"/>
+  <xacro:arg name="robot_command_port" default="1602"/>
+  <xacro:arg name="load_ros2_control" default="false"/>
+  <xacro:arg name="load_hand" default="false"/>
+  <xacro:arg name="use_sim" default="false"/>
+  <xacro:arg name="connected_to" default=""/>
+  <xacro:arg name="xyz" default="0 0 0"/>
+  <xacro:arg name="rpy" default="0 0 0"/>
+  <xacro:include filename="$(find franka_panda_description)/robots/panda_arm.xacro"/>
+  <xacro:panda_arm prefix="$(arg prefix)" connected_to="$(arg connected_to)" xyz="$(arg xyz)" rpy="$(arg rpy)"/>
+  <xacro:if value="$(arg load_ros2_control)">
     <!-- Import ros2_control description -->
     <xacro:include filename="$(find franka_panda_description)/ros2_control/panda_arm.ros2_control.xacro"/>
-    <xacro:panda_arm prefix="$(arg prefix)" connected_to="$(arg connected_to)" xyz="$(arg xyz)" rpy="$(arg rpy)"/>
-    <xacro:if value="$(arg load_ros2_control)">
-        <xacro:panda_arm_interface
-                name="PandaInterface"
-                prefix="$(arg prefix)"
-                robot_ip="$(arg robot_ip)"
-                robot_state_port="$(arg robot_state_port)"
-                robot_command_port="$(arg robot_command_port)"
-                use_sim="$(arg use_sim)"
-        />
-    </xacro:if>
-    <xacro:if value="$(arg load_hand)">
-        <xacro:include filename="$(find franka_panda_description)/robots/hand.xacro"/>
-        <xacro:hand prefix="$(arg prefix)" rpy="0 0 ${-pi/4}" connected_to="$(arg prefix)link8"/>
-    </xacro:if>
+    <xacro:panda_arm_interface
+        name="PandaInterface"
+        prefix="$(arg prefix)"
+        robot_ip="$(arg robot_ip)"
+        robot_state_port="$(arg robot_state_port)"
+        robot_command_port="$(arg robot_command_port)"
+        use_sim="$(arg use_sim)"
+    />
+  </xacro:if>
+  <xacro:if value="$(arg load_hand)">
+    <xacro:include filename="$(find franka_panda_description)/robots/hand.xacro"/>
+    <xacro:hand prefix="$(arg prefix)" connected_to="$(arg prefix)link8" rpy="0 0 ${-pi/4}"/>
+  </xacro:if>
 </robot>

File: robots/panda_arm.xacro (robot description, xacro)
@@ -1,8 +1,8 @@
 <?xml version='1.0'?>
 <robot xmlns:xacro="http://www.ros.org/wiki/xacro" name="panda">
-  <xacro:macro name="panda_arm" params="prefix:='panda_' description_pkg:='franka_panda_description' connected_to:='' in_gazebo='false' xyz:='0 0 0' rpy:='0 0 0'">
+  <xacro:macro name="panda_arm" params="prefix:='panda_' connected_to:='' in_gazebo='false' xyz:='0 0 0' rpy:='0 0 0'">
     <!-- If using custom frame with ${connected_to} param, make sure 'world' frame exists in its TF tree -->
     <xacro:if value="${connected_to == ''}">
-      <link name="world" />
+      <link name="world"/>
       <xacro:property name="base_frame_name" value="world"/>
     </xacro:if>
@@ -21,10 +21,10 @@
       <visual>
         <geometry>
-          <mesh filename="package://${description_pkg}/meshes/visual/link0.dae"/>
-        </geometry>
-      </visual>
-      <collision>
-        <geometry>
-          <mesh filename="package://${description_pkg}/meshes/collision/link0.stl"/>
+          <mesh filename="package://franka_panda_description/meshes/visual/link0.dae"/>
+        </geometry>
+      </visual>
+      <collision>
+        <geometry>
+          <mesh filename="package://franka_panda_description/meshes/collision/link0.stl"/>
         </geometry>
       </collision>
@@ -40,10 +40,10 @@
       <visual>
         <geometry>
-          <mesh filename="package://${description_pkg}/meshes/visual/link1.dae"/>
-        </geometry>
-      </visual>
-      <collision>
-        <geometry>
-          <mesh filename="package://${description_pkg}/meshes/collision/link1.stl"/>
+          <mesh filename="package://franka_panda_description/meshes/visual/link1.dae"/>
+        </geometry>
+      </visual>
+      <collision>
+        <geometry>
+          <mesh filename="package://franka_panda_description/meshes/collision/link1.stl"/>
         </geometry>
       </collision>
@@ -51,5 +51,6 @@
         <origin xyz="3.875e-03 2.081e-03 -0.1750" rpy="0 0 0"/>
         <mass value="4.970684"/>
-        <inertia ixx="7.0337e-01" ixy="-1.3900e-04" ixz="6.7720e-03" iyy="7.0661e-01" iyz="1.9169e-02" izz="9.1170e-03"/>
+        <inertia ixx="7.0337e-01" ixy="-1.3900e-04" ixz="6.7720e-03" iyy="7.0661e-01" iyz="1.9169e-02"
+                 izz="9.1170e-03"/>
       </inertial>
     </link>
@@ -66,10 +67,10 @@
       <visual>
         <geometry>
-          <mesh filename="package://${description_pkg}/meshes/visual/link2.dae"/>
-        </geometry>
-      </visual>
-      <collision>
-        <geometry>
-          <mesh filename="package://${description_pkg}/meshes/collision/link2.stl"/>
+          <mesh filename="package://franka_panda_description/meshes/visual/link2.dae"/>
+        </geometry>
+      </visual>
+      <collision>
+        <geometry>
+          <mesh filename="package://franka_panda_description/meshes/collision/link2.stl"/>
         </geometry>
       </collision>
@@ -77,5 +78,6 @@
         <origin xyz="-3.141e-03 -2.872e-02 3.495e-03" rpy="0 0 0"/>
         <mass value="0.646926"/>
-        <inertia ixx="7.9620e-03" ixy="-3.9250e-03" ixz="1.0254e-02" iyy="2.8110e-02" iyz="7.0400e-04" izz="2.5995e-02"/>
+        <inertia ixx="7.9620e-03" ixy="-3.9250e-03" ixz="1.0254e-02" iyy="2.8110e-02" iyz="7.0400e-04"
+                 izz="2.5995e-02"/>
       </inertial>
     </link>
@@ -92,10 +94,10 @@
       <visual>
         <geometry>
-          <mesh filename="package://${description_pkg}/meshes/visual/link3.dae"/>
-        </geometry>
-      </visual>
-      <collision>
-        <geometry>
-          <mesh filename="package://${description_pkg}/meshes/collision/link3.stl"/>
+          <mesh filename="package://franka_panda_description/meshes/visual/link3.dae"/>
+        </geometry>
+      </visual>
+      <collision>
+        <geometry>
+          <mesh filename="package://franka_panda_description/meshes/collision/link3.stl"/>
         </geometry>
       </collision>
@@ -103,5 +105,6 @@
         <origin xyz="2.7518e-02 3.9252e-02 -6.6502e-02" rpy="0 0 0"/>
         <mass value="3.228604"/>
-        <inertia ixx="3.7242e-02" ixy="-4.7610e-03" ixz="-1.1396e-02" iyy="3.6155e-02" iyz="-1.2805e-02" izz="1.0830e-02"/>
+        <inertia ixx="3.7242e-02" ixy="-4.7610e-03" ixz="-1.1396e-02" iyy="3.6155e-02" iyz="-1.2805e-02"
+                 izz="1.0830e-02"/>
       </inertial>
     </link>
@@ -118,10 +121,10 @@
       <visual>
         <geometry>
-          <mesh filename="package://${description_pkg}/meshes/visual/link4.dae"/>
-        </geometry>
-      </visual>
-      <collision>
-        <geometry>
-          <mesh filename="package://${description_pkg}/meshes/collision/link4.stl"/>
+          <mesh filename="package://franka_panda_description/meshes/visual/link4.dae"/>
+        </geometry>
+      </visual>
+      <collision>
+        <geometry>
+          <mesh filename="package://franka_panda_description/meshes/collision/link4.stl"/>
         </geometry>
       </collision>
@@ -129,5 +132,6 @@
         <origin xyz="-5.317e-02 1.04419e-01 2.7454e-02" rpy="0 0 0"/>
         <mass value="3.587895"/>
-        <inertia ixx="2.5853e-02" ixy="7.7960e-03" ixz="-1.3320e-03" iyy="1.9552e-02" iyz="8.6410e-03" izz="2.8323e-02"/>
+        <inertia ixx="2.5853e-02" ixy="7.7960e-03" ixz="-1.3320e-03" iyy="1.9552e-02" iyz="8.6410e-03"
+                 izz="2.8323e-02"/>
       </inertial>
     </link>
@@ -144,10 +148,10 @@
       <visual>
         <geometry>
-          <mesh filename="package://${description_pkg}/meshes/visual/link5.dae"/>
-        </geometry>
-      </visual>
-      <collision>
-        <geometry>
-          <mesh filename="package://${description_pkg}/meshes/collision/link5.stl"/>
+          <mesh filename="package://franka_panda_description/meshes/visual/link5.dae"/>
+        </geometry>
+      </visual>
+      <collision>
+        <geometry>
+          <mesh filename="package://franka_panda_description/meshes/collision/link5.stl"/>
         </geometry>
       </collision>
@@ -155,5 +159,6 @@
         <origin xyz="-1.1953e-02 4.1065e-02 -3.8437e-02" rpy="0 0 0"/>
         <mass value="1.225946"/>
-        <inertia ixx="3.5549e-02" ixy="-2.1170e-03" ixz="-4.0370e-03" iyy="2.9474e-02" iyz="2.2900e-04" izz="8.6270e-03"/>
+        <inertia ixx="3.5549e-02" ixy="-2.1170e-03" ixz="-4.0370e-03" iyy="2.9474e-02" iyz="2.2900e-04"
+                 izz="8.6270e-03"/>
       </inertial>
     </link>
@@ -170,10 +175,10 @@
       <visual>
         <geometry>
-          <mesh filename="package://${description_pkg}/meshes/visual/link6.dae"/>
-        </geometry>
-      </visual>
-      <collision>
-        <geometry>
-          <mesh filename="package://${description_pkg}/meshes/collision/link6.stl"/>
+          <mesh filename="package://franka_panda_description/meshes/visual/link6.dae"/>
+        </geometry>
+      </visual>
+      <collision>
+        <geometry>
+          <mesh filename="package://franka_panda_description/meshes/collision/link6.stl"/>
         </geometry>
       </collision>
@@ -181,5 +186,6 @@
         <origin xyz="6.0149e-02 -1.4117e-02 -1.0517e-02" rpy="0 0 0"/>
         <mass value="1.666555"/>
-        <inertia ixx="1.9640e-03" ixy="1.0900e-04" ixz="-1.1580e-03" iyy="4.3540e-03" iyz="3.4100e-04" izz="5.4330e-03"/>
+        <inertia ixx="1.9640e-03" ixy="1.0900e-04" ixz="-1.1580e-03" iyy="4.3540e-03" iyz="3.4100e-04"
+                 izz="5.4330e-03"/>
       </inertial>
     </link>
@@ -196,10 +202,10 @@
       <visual>
         <geometry>
-          <mesh filename="package://${description_pkg}/meshes/visual/link7.dae"/>
-        </geometry>
-      </visual>
-      <collision>
-        <geometry>
-          <mesh filename="package://${description_pkg}/meshes/collision/link7.stl"/>
+          <mesh filename="package://franka_panda_description/meshes/visual/link7.dae"/>
+        </geometry>
+      </visual>
+      <collision>
+        <geometry>
+          <mesh filename="package://franka_panda_description/meshes/collision/link7.stl"/>
         </geometry>
       </collision>
@@ -207,5 +213,6 @@
         <origin xyz="1.0517e-02 -4.252e-03 6.1597e-02" rpy="0 0 0"/>
         <mass value="7.35522e-01"/>
-        <inertia ixx="1.2516e-02" ixy="-4.2800e-04" ixz="-1.1960e-03" iyy="1.0027e-02" iyz="-7.4100e-04" izz="4.8150e-03"/>
+        <inertia ixx="1.2516e-02" ixy="-4.2800e-04" ixz="-1.1960e-03" iyy="1.0027e-02" iyz="-7.4100e-04"
+                 izz="4.8150e-03"/>
       </inertial>
     </link>
@@ -227,5 +234,5 @@
     </link>
     <joint name="${prefix}joint8" type="fixed">
-    <origin rpy="0 0 0" xyz="0 0 0.107"/>
+      <origin rpy="0 0 0" xyz="0 0 0.107"/>
       <parent link="${prefix}link7"/>
       <child link="${prefix}link8"/>

File: robots/panda_arm_hand_cam.urdf.xacro (robot description, xacro)
@@ -5,5 +5,4 @@
   <xacro:arg name="robot_state_port" default="1601"/>
   <xacro:arg name="robot_command_port" default="1602"/>
-  <xacro:arg name="load_gazebo" default="false"/>
   <xacro:arg name="load_ros2_control" default="false"/>
   <xacro:arg name="use_sim" default="false"/>
@@ -11,17 +10,17 @@
   <xacro:arg name="xyz" default="0 0 0"/>
   <xacro:arg name="rpy" default="0 0 0"/>
-  <!-- Import ros2_control description -->
-  <xacro:include filename="$(find franka_panda_description)/ros2_control/panda_arm.ros2_control.xacro"/>
   <xacro:include filename="$(find franka_panda_description)/robots/panda_arm.xacro"/>
-  <xacro:include filename="$(find franka_panda_description)/robots/hand.xacro"/>
+  <xacro:panda_arm prefix="$(arg prefix)" connected_to="$(arg connected_to)" xyz="$(arg xyz)" rpy="$(arg rpy)"/>
   <xacro:include filename="$(find franka_panda_description)/robots/l515_adapter.xacro"/>
+  <xacro:l515_adapter prefix="$(arg prefix)holder_" connected_to="$(arg prefix)link8" rpy="0 0 ${-pi/4}"/>
   <xacro:include filename="$(find realsense2_description)/urdf/_l515.urdf.xacro"/>
-  <xacro:panda_arm prefix="$(arg prefix)" connected_to="$(arg connected_to)" xyz="$(arg xyz)" rpy="$(arg rpy)"/>
-  <xacro:l515_adapter prefix="$(arg prefix)holder_" connected_to="$(arg prefix)link8" rpy="0 0 ${-pi/4}"/>
   <xacro:sensor_l515 parent="$(arg prefix)holder_cam" use_nominal_extrinsics="true" add_plug="true" use_mesh="false">
     <origin xyz="0 -0.03015 0.014" rpy="${-pi/2} ${-pi/2} 0"/>
   </xacro:sensor_l515>
+  <xacro:include filename="$(find franka_panda_description)/robots/hand.xacro"/>
   <xacro:hand prefix="$(arg prefix)" connected_to="$(arg prefix)holder_toolside"/>
   <xacro:if value="$(arg load_ros2_control)">
+    <!-- Import ros2_control description -->
+    <xacro:include filename="$(find franka_panda_description)/ros2_control/panda_arm.ros2_control.xacro"/>
     <xacro:panda_arm_interface
         name="PandaInterface"
