Commit message: fix: remove the _ and put it in prefix

File: ros2_control/panda_arm.ros2_control.xacro (robot description, xacro)
@@ -1,10 +1,10 @@
 <?xml version="1.0"?>
 <robot xmlns:xacro="http://www.ros.org/wiki/xacro">
-  <xacro:macro name="panda_arm_interface" params="name prefix:='panda'">
+  <xacro:macro name="panda_arm_interface" params="name prefix:='panda_'">
     <ros2_control name="${name}" type="system">
       <hardware>
         <plugin>robot_interface/franka/PandaInterface</plugin>
       </hardware>
-      <joint name="${prefix}_joint1">
+      <joint name="${prefix}joint1">
         <command_interface name="position">
           <param name="min">-2.8973</param>
@@ -24,5 +24,5 @@
         <state_interface name="effort"/>
       </joint>
-      <joint name="${prefix}_joint2">
+      <joint name="${prefix}joint2">
         <command_interface name="position">
           <param name="min">-1.7628</param>
@@ -42,5 +42,5 @@
         <state_interface name="effort"/>
       </joint>
-      <joint name="${prefix}_joint3">
+      <joint name="${prefix}joint3">
         <command_interface name="position">
           <param name="min">-2.8973</param>
@@ -60,5 +60,5 @@
         <state_interface name="effort"/>
       </joint>
-      <joint name="${prefix}_joint4">
+      <joint name="${prefix}joint4">
         <command_interface name="position">
           <param name="min">-3.0718</param>
@@ -78,5 +78,5 @@
         <state_interface name="effort"/>
       </joint>
-      <joint name="${prefix}_joint5">
+      <joint name="${prefix}joint5">
         <command_interface name="position">
           <param name="min">-2.8973</param>
@@ -96,5 +96,5 @@
         <state_interface name="effort"/>
       </joint>
-      <joint name="${prefix}_joint6">
+      <joint name="${prefix}joint6">
         <command_interface name="position">
           <param name="min">-0.0175</param>
@@ -114,5 +114,5 @@
         <state_interface name="effort"/>
       </joint>
-      <joint name="${prefix}_joint7">
+      <joint name="${prefix}joint7">
         <command_interface name="position">
           <param name="min">-2.8973</param>

Commit message: feat: add simulation tag

File: ros2_control/panda_arm.ros2_control.xacro (robot description, xacro)
@@ -1,8 +1,13 @@
 <?xml version="1.0"?>
 <robot xmlns:xacro="http://www.ros.org/wiki/xacro">
-  <xacro:macro name="panda_arm_interface" params="name prefix:='panda_'">
+  <xacro:macro name="panda_arm_interface" params="name prefix:='panda_' use_sim:=^|false">
     <ros2_control name="${name}" type="system">
       <hardware>
-        <plugin>robot_interface/franka/PandaInterface</plugin>
+        <xacro:if value="$(arg use_sim)">
+          <plugin>robot_interface/simulators/PybulletInterface</plugin>
+        </xacro:if>
+        <xacro:unless value="$(arg use_sim)">
+          <plugin>robot_interface/franka/PandaInterface</plugin>
+        </xacro:unless>
       </hardware>
       <joint name="${prefix}joint1">

Commit message: Add communication parameters in the URDF (#6)
* fix: correct the quote typo

File: ros2_control/panda_arm.ros2_control.xacro (robot description, xacro)
@@ -1,14 +1,20 @@
 <?xml version="1.0"?>
 <robot xmlns:xacro="http://www.ros.org/wiki/xacro">
-  <xacro:macro name="panda_arm_interface" params="name prefix use_sim:=^|false">
+  <xacro:macro name="panda_arm_interface" params="name prefix robot_ip robot_state_port robot_command_port use_sim">
     <ros2_control name="${name}" type="system">
-      <xacro:if value="$(arg use_sim)">
+      <xacro:if value="${use_sim}">
         <hardware>
           <plugin>robot_interface/simulators/PybulletInterface</plugin>
+          <param name="robot_ip">${robot_ip}</param>
+          <param name="robot_state_port">${robot_state_port}</param>
+          <param name="robot_command_port">${robot_command_port}</param>
         </hardware>
       </xacro:if>
-      <xacro:unless value="$(arg use_sim)">
+      <xacro:unless value="${use_sim}">
         <hardware>
           <plugin>robot_interface/franka/PandaInterface</plugin>
+          <param name="robot_ip">${robot_ip}</param>
+          <param name="robot_state_port">${robot_state_port}</param>
+          <param name="robot_command_port">${robot_command_port}</param>
         </hardware>
       </xacro:unless>
